File: corne-ultralight/pcb/corne-ultralight.kicad_pcb (KiCad board)
At the start: 2 copper layers, 275.5 x 105.6 mm, 132 parts, among them J2 OLED, J5 Breakaway_Tabs, J7 OLED, SW1 SW_PUSH, SW10 SW_PUSH, SW11 SW_PUSH, SW12 SW_PUSH, SW13 SW_PUSH, SW14 SW_PUSH, SW15 SW_PUSH, SW16 SW_PUSH, SW17 SW_PUSH, SW18 SW_PUSH, SW19 SW_PUSH, SW2 SW_PUSH, SW20 SW_PUSH, SW21 SW_PUSH, SW22 SW_PUSH, SW23 SW_PUSH, SW24 SW_PUSH, SW25 SW_PUSH, SW26 SW_PUSH, SW27 SW_PUSH, SW28 SW_PUSH, SW29 SW_PUSH, SW3 SW_PUSH, SW30 SW_PUSH, SW31 SW_PUSH, SW32 SW_PUSH, SW33 SW_PUSH, SW34 SW_PUSH, SW35 SW_PUSH, SW36 SW_PUSH, SW37 SW_PUSH, SW38 SW_PUSH, SW39 SW_PUSH, SW4 SW_PUSH, SW40 SW_PUSH, SW41 SW_PUSH, SW42 SW_PUSH, SW5 SW_PUSH, SW6 SW_PUSH, SW7 SW_PUSH, SW8 SW_PUSH, SW9 SW_PUSH, U1 xiao-ble, U2 ProMicro

Commit message: Left side completed
Parts:
- removed TP1: RGB, TestPoint:TestPoint_Pad_D1.5mm
- moved TP3 51.0 mm to (136.9, 95.8)
- moved TP2 48.7 mm to (140.4, 97.2)
Routing:
- net col5: track 114.5 -> 139.6 mm, vias 8 -> 12
- net row0: track 156.0 -> 131.8 mm
- net Net-(BATJ1-Pad2): track 33.1 -> 13.1 mm, vias 1 -> 0
- net RGB: track 19.3 -> 0.00 mm
- net col2: track 141.2 -> 158.8 mm, vias 7 -> 8
- net col4: track 138.9 -> 156.2 mm, vias 8 -> 9
- net GND: track 88.9 -> 72.2 mm, vias 0 -> 1
- net col3: track 153.5 -> 169.8 mm, vias 8 -> 9
- net VCC: track 43.1 -> 58.7 mm, vias 0 -> 3
- net row1: track 175.5 -> 161.0 mm
- net col1: track 166.0 -> 175.5 mm, vias 7 -> 10
- net +5V: track 0.00 -> 7.29 mm
- net reset: track 50.1 -> 43.4 mm, vias 0 -> 1
- net col0: track 187.9 -> 193.3 mm, vias 8 -> 11
- net CS: track 35.4 -> 31.2 mm, vias 0 -> 2
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
Commit message: update footptint
Parts:
- TP4: moved to F.Cu
- U2: value ProMicro -> xiao-ble; footprint kbd:ProMicro_v3 -> kleeb-mcu:xiao-ble-tht
- moved TP4 192.1 mm to (1.27, 1.27), turned to 0 degrees
- moved U2 6.85 mm to (164.0, 49.8)
Connections:
- U1 pad 12: VCC -> unconnected-(U1-3V3-Pad12)
- U1 pad 14: +BATT -> unconnected-(U1-5V-Pad14)
- U1 pad 19: unconnected-(U1-Pad19) -> +BATT
- U2 pad 1: RGB_r -> row0_r
- U2 pad 10: row3_r -> col3_r
- U2 pad 11: unconnected-(U2-Pad11) -> col2_r
- U2 pad 13: unconnected-(U2-Pad13) -> GNDA
- U2 pad 15: col5_r -> unconnected-(U2-A31_SWDIO-Pad15)
- U2 pad 16: col4_r -> unconnected-(U2-A30_SWCLK-Pad16)
- U2 pad 17: col3_r -> reset_r
- U2 pad 18: col2_r -> GNDA
- U2 pad 19: col1_r -> +BATTA
- U2 pad 2: CS_r -> row1_r
- U2 pad 20: col0_r -> GNDA
- U2 pad 21: VDD -> col1_r
- U2 pad 22: reset_r -> col0_r
- U2 pad 3: GNDA -> row2_r
- U2 pad 4: GNDA -> row3_r
- U2 pad 7: row0_r -> CS_r
- U2 pad 8: row1_r -> col5_r
- U2 pad 9: row2_r -> col4_r
Routing:
- net RGB_r: track 55.8 -> 0.00 mm, vias 1 -> 0
- net reset_r: track 79.7 -> 41.6 mm, vias 0 -> 4
- net VCC: track 58.7 -> 21.5 mm, vias 3 -> 1
- net row3_r: track 81.6 -> 109.9 mm, vias 3 -> 4
- net row0_r: track 143.3 -> 171.6 mm, vias 12 -> 11
- net row1_r: track 148.9 -> 174.0 mm
- net row2_r: track 155.2 -> 178.3 mm
- net VDD: track 54.3 -> 31.8 mm
- net col5_r: track 123.6 -> 102.8 mm
- net col0_r: track 203.1 -> 191.0 mm
- net col4_r: track 140.0 -> 150.8 mm, vias 2 -> 3
- net col3_r: track 165.1 -> 175.6 mm, vias 4 -> 5
- net col2_r: track 157.2 -> 167.0 mm, vias 3 -> 4
- net col1_r: track 175.0 -> 166.1 mm
- net CS_r: track 35.2 -> 26.9 mm, vias 0 -> 2
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Other:
- board text added: "rev 3x"
- board text removed: "rev 2.1"
